File: Jupiter/Astro Boost.kicad_sch (KiCad schematic)
At the start: 34 parts, among them J1 AudioJack2, J10 Power from SW to PS, J2 AudioJack2, J3 Jack-DC, J4 Signal In, J5 Audio In, J6 Processed to SW, J7 Bypass, J8 Processed Out, J9 Power from 9V to SW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

Commit message: updated fix it list
Other:
- note added: "double check all components, link datasheets and part numbers"
- note removed: "link datasheets"
Changed lines of the file:
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@@
 		)
 	)
-	(text "link datasheets"
+	(text "double check all components, link datasheets and part numbers"
 		(exclude_from_sim no)
 		(at 236.982 81.026 0)

Commit message: Updates to Saturn
Removed wiring pads and associated tracks
Added to do list
Shortened PCB
Other:
- note added: "Add a logo and text and stuff"
Changed lines of the file:
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@@
+		)
+	)
+	(text "Add a logo and text and stuff"
+		(exclude_from_sim no)
+		(at 239.776 88.138 0)
+		(effects
+			(font
+				(size 1.27 1.27)
+			)
 		)
 	)
