File: Saturn/Astro Boost.kicad_sch (KiCad schematic)
At the start: 36 parts, among them J1 AudioJack2, J10 Power from SW to PS, J11 +9V, J12 -9V, J2 AudioJack2, J3 Jack-DC, J4 Signal In, J5 Audio In, J6 Processed to SW, J7 Bypass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

Commit message: updates to saturn
layout
Other:
- note added: "Widened r4, r5 and r2 made U1 more Narrow Updated r3 from .8mm hole size to 1mm hole size"
- note removed: "Widened r4, r5 and r2"
Changed lines of the file:
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@@
 		)
 	)
-	(text "Widened r4, r5 and r2"
+	(text "Widened r4, r5 and r2\nmade U1 more Narrow\nUpdated r3 from .8mm hole size to 1mm hole size"
 		(exclude_from_sim no)
-		(at 249.936 121.412 0)
+		(at 248.666 124.968 0)
 		(effects
 			(font

Commit message: Updates to saturn
Parts:
- C1, C5: footprint Capacitor_THT:C_Disc_D9.0mm_W5.0mm_P10.00mm -> Capacitor_THT:C_Axial_L12.0mm_D6.5mm_P20.00mm_Horizontal
- C2, C4: footprint Capacitor_THT:C_Disc_D9.0mm_W5.0mm_P10.00mm -> Capacitor_THT:C_Axial_L12.0mm_D9.5mm_P20.00mm_Horizontal
Changed lines of the file:
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@@
 			)
 		)
-		(property "Footprint" "Capacitor_THT:C_Disc_D9.0mm_W5.0mm_P10.00mm"
+		(property "Footprint" "Capacitor_THT:C_Axial_L12.0mm_D9.5mm_P20.00mm_Horizontal"
 			(at 152.4 89.8652 0)
 			(effects
@@
 			)
 		)
-		(property "Datasheet" "~"
+		(property "Datasheet" "https://www.mouser.com/datasheet/2/449/Elytone_23P_Series-3182363.pdf"
 			(at 156.21 88.9 0)
 			(effects
@@
 			)
 		)
-		(property "Description" "564R30GAS10"
+		(property "Description" "23PS310"
 			(at 156.21 88.9 0)
 			(effects
@@
 			)
 		)
-		(property "Footprint" "Capacitor_THT:C_Disc_D9.0mm_W5.0mm_P10.00mm"
+		(property "Footprint" "Capacitor_THT:C_Axial_L12.0mm_D6.5mm_P20.00mm_Horizontal"
 			(at 100.33 88.5952 0)
 			(effects
@@
 			)
 		)
-		(property "Description" "S502M75Z5UR83L0R"
+		(property "Description" "23PS250"
 			(at 104.14 87.63 0)
 			(effects
@@
 			)
 		)
-		(property "Footprint" "Capacitor_THT:C_Disc_D9.0mm_W5.0mm_P10.00mm"
+		(property "Footprint" "Capacitor_THT:C_Axial_L12.0mm_D9.5mm_P20.00mm_Horizontal"
 			(at 100.33 93.6752 0)
 			(effects
@@
 			)
 		)
-		(property "Datasheet" "~"
+		(property "Datasheet" "https://www.mouser.com/datasheet/2/449/Elytone_23P_Series-3182363.pdf"
 			(at 104.14 92.71 0)
 			(effects
@@
 			)
 		)
-		(property "Description" "564R30GAS10"
+		(property "Description" "23PS310"
 			(at 104.14 92.71 0)
 			(effects
@@
 			)
 		)
-		(property "Footprint" "Capacitor_THT:C_Disc_D9.0mm_W5.0mm_P10.00mm"
+		(property "Footprint" "Capacitor_THT:C_Axial_L12.0mm_D6.5mm_P20.00mm_Horizontal"
 			(at 100.33 101.2952 0)
 			(effects
@@
 			)
 		)
-		(property "Description" "S502M75Z5UR83L0R"
+		(property "Description" "23PS250"
 			(at 104.14 100.33 0)
 			(effects
